File: WIFIAdapter.sch (EAGLE design)
At the start: 17 parts

Commit message: RevE with 8 pin DIP adapter
Trade the break away PCB adapter for a COTS ribbon cable DIP adapter.
Parts:
- removed JP3, JP4: (no value), SparkFun-Connectors:M03X2SHROUD
- removed JP5, JP6: (no value), SparkFun-Connectors:M04LOCK
- removed JP7: (no value), SparkFun-Connectors:M03LOCK
- removed STANDOFF3: STAND-OFFTIGHT, SparkFun-Electromechanical:STAND-OFFTIGHT
- added S1: (no value), SparkFun-Electromechanical:TAC_SWITCHPTH
- added U$1: M04X2, SparkFun-Connectors:M04X2
Connections:
- net N$1 renamed TX
- net N$2 renamed RX
- removed net N$10: JP3.5, JP6.4
- removed net N$12: JP3.4, JP5.4
- removed net N$4: JP3.1, JP6.1
- removed net N$5: JP3.2, JP6.3
- removed net N$6: JP7.3, U$2.4
- removed net N$9: JP3.3, JP6.2
- net 5V: now also U$1.1; no longer JP4.1
- net GND: now also S1.3, S1.4, U$1.7; no longer JP4.5, JP7.2
- net N$11: now also U$1.2; no longer JP4.4
- net N$7: now also S1.1, S1.2; no longer JP7.1
Other:
- note added: "E"
- note removed: "D"
